Commit message: finished robot structure, added lidar, and modified the launch file in accordance!

File: urdf/barista_robot_model.urdf (robot description, URDF)
Before this commit: robot box_bot, 9 links, 8 joints
Links:
- added link back_caster_wheel, mass 0.05; collision sphere radius=0.0352; visual sphere radius=0.0352
- added link front_caster_wheel, mass 0.05; collision sphere radius=0.0352; visual sphere radius=0.0352
- added link laser_scanner, mass 0.01; collision cylinder length=0.0408 radius=0.037493; visual mesh filename=package://barista_robot_description/meshes/sick_microscan3.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 scale=0.5 0.5 0.5
- link chassis: mass None -> 1.5; geometry collision cylinder length=0.155 radius=0.178; visual cylinder length=0.155 radius=0.178
- link left_wheel: mass None -> 0.2; geometry collision cylinder length=0.0206 radius=0.0352; visual cylinder length=0.0206 radius=0.0352
- link right_wheel: mass None -> 0.2; geometry collision cylinder length=0.0206 radius=0.0352; visual cylinder length=0.0206 radius=0.0352
- link standoff_rod_1: mass None -> 0.1; geometry collision cylinder length=0.220 radius=0.010; visual cylinder length=0.220 radius=0.010
- link standoff_rod_2: mass None -> 0.1; geometry collision cylinder length=0.220 radius=0.010; visual cylinder length=0.220 radius=0.010
- link standoff_rod_3: mass None -> 0.1; geometry collision cylinder length=0.220 radius=0.010; visual cylinder length=0.220 radius=0.010
- link standoff_rod_4: mass None -> 0.1; geometry collision cylinder length=0.220 radius=0.010; visual cylinder length=0.220 radius=0.010
- link tray: mass None -> 0.5; geometry collision cylinder length=0.090 radius=0.160; visual cylinder length=0.090 radius=0.160
Joints:
- added joint back_pitch_joint: type continuous, parent chassis, child back_caster_wheel, origin xyz=-0.140 0 -0.0775 rpy=0 0 0, axis 0 1 0, limit effort=1000.0 velocity=100.0
- added joint front_pitch_joint: type continuous, parent chassis, child front_caster_wheel, origin xyz=0.140 0 -0.0775 rpy=0 0 0, axis 0 1 0, limit effort=1000.0 velocity=100.0
- added joint joint_laser_scanner: type continuous, parent chassis, child laser_scanner, origin xyz=0.120 0.0 0.1 rpy=0 0 0, axis 0 0 1, limit effort=10.0 velocity=2.0
- joint joint_standoff_rod_1: origin xyz=0 0.140 0.1875 rpy=0 0 0 -> xyz=0.100 0.100 0.1875 rpy=0 0 0
- joint joint_standoff_rod_2: origin xyz=0 -0.140 0.1875 rpy=0 0 0 -> xyz=0.100 -0.100 0.1875 rpy=0 0 0
- joint joint_standoff_rod_3: origin xyz=-0.140 0 0.1875 rpy=0 0 0 -> xyz=-0.100 -0.100 0.1875 rpy=0 0 0
- joint joint_standoff_rod_4: origin xyz=0.140 0 0.1875 rpy=0 0 0 -> xyz=-0.100 0.100 0.1875 rpy=0 0 0

Commit message: xacrofied model of the barista robot and created tag task2 !

File: urdf/barista_robot_model.urdf (robot description, URDF)
Before this commit: robot barista_bot, 12 links, 11 joints
Links:
- link back_caster_wheel: geometry collision sphere radius=${caster_radius}; visual sphere radius=${caster_radius}
- link chassis: mass 1.5 -> ${chassis_mass}; geometry collision cylinder length=${chassis_length} radius=${chassis_radius}; visual cylinder length=${chassis_length} radius=${chassis_radius}
- link front_caster_wheel: geometry collision sphere radius=${caster_radius}; visual sphere radius=${caster_radius}
- link left_wheel: mass 0.2 -> ${wheel_mass}; geometry collision cylinder length=${wheel_length} radius=${wheel_radius}; visual cylinder length=${wheel_length} radius=${wheel_radius}
- link right_wheel: mass 0.2 -> ${wheel_mass}; geometry collision cylinder length=${wheel_length} radius=${wheel_radius}; visual cylinder length=${wheel_length} radius=${wheel_radius}
- link standoff_rod_1: mass 0.1 -> ${rod_mass}; geometry collision cylinder length=${rod_length} radius=${rod_radius}; visual cylinder length=${rod_length} radius=${rod_radius}
- link standoff_rod_2: geometry collision cylinder length=0.220 radius=0.010; visual cylinder length=${rod_length} radius=${rod_radius}
- link standoff_rod_3: mass 0.1 -> ${rod_mass}; geometry collision cylinder length=${rod_length} radius=${rod_radius}; visual cylinder length=${rod_length} radius=${rod_radius}
- link standoff_rod_4: mass 0.1 -> ${rod_mass}; geometry collision cylinder length=${rod_length} radius=${rod_radius}; visual cylinder length=${rod_length} radius=${rod_radius}
- link tray: mass 0.5 -> ${tray_mass}; geometry collision cylinder length=${tray_length} radius=${tray_radius}; visual cylinder length=${tray_length} radius=${tray_radius}
Joints:
- joint back_pitch_joint: origin xyz=-0.140 0 -0.0775 rpy=0 0 0 -> xyz=-${caster_wheel_offset} 0 ${wheel_z_offset} rpy=0 0 0
- joint base_link_joint: origin xyz=0 0 0.1127 rpy=0 0 0 -> xyz=0 0 ${base_link_z} rpy=0 0 0
- joint front_pitch_joint: origin xyz=0.140 0 -0.0775 rpy=0 0 0 -> xyz=${caster_wheel_offset} 0 ${wheel_z_offset} rpy=0 0 0
- joint joint_laser_scanner: origin xyz=0.120 0.0 0.1 rpy=0 0 0 -> xyz=${laser_scanner_origin_xy} 0 ${laser_scanner_origin_z} rpy=0 0 0
- joint joint_left_wheel: origin xyz=0 0.140 -0.0775 rpy=0 0 0 -> xyz=0 ${wheel_y_offset} ${wheel_z_offset} rpy=0 0 0
- joint joint_right_wheel: origin xyz=0 -0.140 -0.0775 rpy=0 0 0 -> xyz=0 -${wheel_y_offset} ${wheel_z_offset} rpy=0 0 0
- joint joint_standoff_rod_1: origin xyz=0.100 0.100 0.1875 rpy=0 0 0 -> xyz=${rod_offset_xy} ${rod_offset_xy} ${rod_z} rpy=0 0 0
- joint joint_standoff_rod_2: origin xyz=0.100 -0.100 0.1875 rpy=0 0 0 -> xyz=${rod_offset_xy} -${rod_offset_xy} ${rod_z} rpy=0 0 0
- joint joint_standoff_rod_3: origin xyz=-0.100 -0.100 0.1875 rpy=0 0 0 -> xyz=-${rod_offset_xy} -${rod_offset_xy} ${rod_z} rpy=0 0 0
- joint joint_standoff_rod_4: origin xyz=-0.100 0.100 0.1875 rpy=0 0 0 -> xyz=-${rod_offset_xy} ${rod_offset_xy} ${rod_z} rpy=0 0 0
- joint joint_tray: origin xyz=0 0 0.3425 rpy=0 0 0 -> xyz=0 0 ${tray_z} rpy=0 0 0

Commit message: corrections of task1 and task2 for tutor evaluation !

File: urdf/barista_robot_model.urdf (robot description, URDF)
Before this commit: robot barista_bot, 12 links, 11 joints
Joints:
- joint joint_standoff_rod_1: origin xyz=${rod_offset_xy} ${rod_offset_xy} ${rod_z} rpy=0 0 0 -> xyz=${rod_offset_x} ${rod_offset_y} ${rod_z} rpy=0 0 0
- joint joint_standoff_rod_2: origin xyz=${rod_offset_xy} -${rod_offset_xy} ${rod_z} rpy=0 0 0 -> xyz=${rod_offset_x} -${rod_offset_y} ${rod_z} rpy=0 0 0
- joint joint_standoff_rod_3: origin xyz=-${rod_offset_xy} -${rod_offset_xy} ${rod_z} rpy=0 0 0 -> xyz=-${rod_offset_x} -${rod_offset_y} ${rod_z} rpy=0 0 0
- joint joint_standoff_rod_4: origin xyz=-${rod_offset_xy} ${rod_offset_xy} ${rod_z} rpy=0 0 0 -> xyz=-${rod_offset_x} ${rod_offset_y} ${rod_z} rpy=0 0 0

File: xacro/barista_very_simple_main.xacro (robot description, xacro)
@@ -72,14 +72,14 @@
   <!-- standoff rods -->
   <xacro:standoff_rod suffix="1" parent="chassis">
-    <origin xyz="0.100 -0.100 0.1875" rpy="0 0 0" />
+    <origin xyz="0.075 -0.100 0.1875" rpy="0 0 0" />
   </xacro:standoff_rod>
   <xacro:standoff_rod suffix="2" parent="chassis">
-    <origin xyz="-0.100 -0.100 0.1875" rpy="0 0 0" />
+    <origin xyz="-0.075 -0.100 0.1875" rpy="0 0 0" />
   </xacro:standoff_rod>
   <xacro:standoff_rod suffix="3" parent="chassis">
-    <origin xyz="-0.100 0.100 0.1875" rpy="0 0 0" />
+    <origin xyz="-0.075 0.100 0.1875" rpy="0 0 0" />
   </xacro:standoff_rod>
   <xacro:standoff_rod suffix="4" parent="chassis">
-    <origin xyz="0.100 0.100 0.1875" rpy="0 0 0" />
+    <origin xyz="0.075 0.100 0.1875" rpy="0 0 0" />
   </xacro:standoff_rod>
   <!-- cup holder tray -->
@@ -98,12 +98,12 @@
   <!-- caster Wheels -->
   <xacro:caster_wheel prefix="front" parent="chassis">
-    <origin xyz="0.140 0 -0.0775" rpy="0 0 0" />
+    <origin xyz="0.110 0 -0.0775" rpy="0 0 0" />
   </xacro:caster_wheel>
   <xacro:caster_wheel prefix="back" parent="chassis">
-    <origin xyz="-0.140 0 -0.0775" rpy="0 0 0" />
+    <origin xyz="-0.110 0 -0.0775" rpy="0 0 0" />
   </xacro:caster_wheel>
   <!-- Laser model -->
   <xacro:laser_scanner parent="chassis">
-    <origin xyz="0.12 0 0.1" rpy="0 0 0" />
+    <origin xyz="0.12 0 0.14" rpy="0 0 0" />
   </xacro:laser_scanner>
   <!-- Gazebo materials -->

File: xacro/laser_scanner.xacro (robot description, xacro)
@@ -11,5 +11,5 @@
       <link name="laser_scanner">
         <visual>
-          <origin rpy="0 0 0" xyz="0 0 -0.0225" />
+          <origin rpy="0 0 0" xyz="0 0 -0.062" />
           <geometry>
             <mesh
@@ -19,5 +19,5 @@
         </visual>
         <collision>
-          <origin rpy="0 0 0" xyz="0 0 0.0204" />
+          <origin rpy="0 0 0" xyz="0 0 -0.062" />
           <geometry>
             <cylinder length="0.0408" radius="0.037493" />
@@ -26,5 +26,5 @@
         <inertial>
           <mass value="0.01" />
-          <origin rpy="0 0 0" xyz="0 0 0.0204" />
+          <origin rpy="0 0 0" xyz="0 0 -0.062" />
           <inertia
             ixx="6.066578520833334e-06"
