Commit message: returned to 1 robot spawn but with manually putting namespace before every frame and robot_description topic

File: xacro/TEST_BARISTA.xacro (robot description, xacro)
@@ -1,4 +1,6 @@
 <?xml version="1.0"?>
 <robot xmlns:xacro="http://www.ros.org/wiki/xacro" name="barista_bot">
+  <xacro:arg name="robot_name" default="barista_X"/>
+  <xacro:property name="robot_name" value="yeyeyea"/>
   <!-- General properties -->
   <xacro:property name="PI" value="3.14159265359"/>
@@ -10,26 +12,13 @@
   <xacro:property name="base_link_z" value="0.1127" /> <!-- length_chassis/2 + wheel_offset -->
   <!-- Standoff rod properties -->
-  <xacro:property name="rod_length" value="0.220" />
-  <xacro:property name="rod_radius" value="0.010" />
-  <xacro:property name="rod_mass" value="0.1" />
-  <xacro:property name="rod_offset_xy" value="0.100" />
-  <xacro:property name="rod_z" value="0.1875" /> <!-- length_rod/2 + length_chassis/2 + wheel_offset -->
+  <xacro:include filename="$(find barista_robot_description)/xacro/standoff_rod.xacro" />
   <!-- Tray properties -->
-  <xacro:property name="tray_length" value="0.090" />
-  <xacro:property name="tray_radius" value="0.160" />
-  <xacro:property name="tray_mass" value="0.5" />
-  <xacro:property name="tray_z" value="0.3425" /><!-- length_tray/2 + length_chassis/2 +  length_rod -->
+  <xacro:include filename="$(find barista_robot_description)/xacro/cup_holder_tray.xacro" />
   <!-- Wheel properties -->
-  <xacro:property name="wheel_length" value="0.0206" />
-  <xacro:property name="wheel_radius" value="0.0352" />
-  <xacro:property name="wheel_mass" value="0.2" />
-  <xacro:property name="wheel_y_offset" value="0.140" />
-  <xacro:property name="wheel_z_offset" value="-0.0775" />
-    <!-- Caster Wheel properties -->
-  <xacro:property name="caster_radius" value=" 0.0352" />
-  <xacro:property name="caster_wheel_offset" value="0.140" />
+  <xacro:include filename="$(find barista_robot_description)/xacro/drive_wheel.xacro" />
+  <!-- Caster Wheel properties -->
+  <xacro:include filename="$(find barista_robot_description)/xacro/caster_wheel.xacro" />
   <!-- laser property -->
-  <xacro:property name="laser_scanner_origin_z" value="0.1"/>
-  <xacro:property name="laser_scanner_origin_xy" value="0.12"/>
+  <xacro:include filename="$(find barista_robot_description)/xacro/laser_scanner.xacro" />
   <!-- Material properties -->
   <xacro:property name="light_gray_color" value="0.8 0.8 0.8 1" />
@@ -84,273 +73,40 @@
   </joint>
   <!-- standoff rods -->
-  <link name="standoff_rod_1">
-    <visual>
-      <geometry>
-        <cylinder length="${rod_length}" radius="${rod_radius}" />
-      </geometry>
-      <material name="light_gray" />
-    </visual>
-    <collision>
-      <geometry>
-        <cylinder length="${rod_length}" radius="${rod_radius}" />
-      </geometry>
-    </collision>
-    <inertial>
-      <origin rpy="0 0 0" xyz="0 0 0" />
-      <mass value="${rod_mass}" />
-      <inertia ixx="0.0001" iyy="0.0001" izz="0.0001" ixy="0.0" ixz="0.0"
-        iyz="0.0" />
-    </inertial>
-  </link>
-  <link name="standoff_rod_2">
-    <visual>
-      <geometry>
-        <cylinder length="${rod_length}" radius="${rod_radius}" />
-      </geometry>
-      <material name="light_gray" />
-    </visual>
-    <collision>
-      <geometry>
-        <cylinder length="0.220" radius="0.010" />
-      </geometry>
-    </collision>
-    <inertial>
-      <origin rpy="0 0 0" xyz="0 0 0" />
-      <mass value="0.1" />
-      <inertia ixx="0.0001" iyy="0.0001" izz="0.0001" ixy="0.0" ixz="0.0"
-        iyz="0.0" />
-    </inertial>
-  </link>
-  <link name="standoff_rod_3">
-    <visual>
-      <geometry>
-        <cylinder length="${rod_length}" radius="${rod_radius}" />
-      </geometry>
-      <material name="light_gray" />
-    </visual>
-    <collision>
-      <geometry>
-        <cylinder length="${rod_length}" radius="${rod_radius}" />
-      </geometry>
-    </collision>
-    <inertial>
-      <origin rpy="0 0 0" xyz="0 0 0" />
-      <mass value="${rod_mass}" />
-      <inertia ixx="0.0001" iyy="0.0001" izz="0.0001" ixy="0.0" ixz="0.0"
-        iyz="0.0" />
-    </inertial>
-  </link>
-  <link name="standoff_rod_4">
-    <visual>
-      <geometry>
-        <cylinder length="${rod_length}" radius="${rod_radius}" />
-      </geometry>
-      <material name="light_gray" />
-    </visual>
-    <collision>
-      <geometry>
-        <cylinder length="${rod_length}" radius="${rod_radius}" />
-      </geometry>
-    </collision>
-    <inertial>
-      <origin rpy="0 0 0" xyz="0 0 0" />
-      <mass value="${rod_mass}" />
-      <inertia ixx="0.0001" iyy="0.0001" izz="0.0001" ixy="0.0" ixz="0.0"
-        iyz="0.0" />
-    </inertial>
-  </link>
-  <joint name="joint_standoff_rod_1" type="fixed">
-    <origin rpy="0 0 0" xyz="${rod_offset_xy} ${rod_offset_xy} ${rod_z}" />
-    <parent link="chassis" />
-    <child link="standoff_rod_1" />
-  </joint>
-  <joint name="joint_standoff_rod_2" type="fixed">
-    <origin rpy="0 0 0" xyz="${rod_offset_xy} -${rod_offset_xy} ${rod_z}" />
-    <parent link="chassis" />
-    <child link="standoff_rod_2" />
-  </joint>
-  <joint name="joint_standoff_rod_3" type="fixed">
-    <origin rpy="0 0 0" xyz="-${rod_offset_xy} -${rod_offset_xy} ${rod_z}" />
-    <parent link="chassis" />
-    <child link="standoff_rod_3" />
-  </joint>
-  <joint name="joint_standoff_rod_4" type="fixed">
-    <origin rpy="0 0 0" xyz="-${rod_offset_xy} ${rod_offset_xy} ${rod_z}" />
-    <parent link="chassis" />
-    <child link="standoff_rod_4" />
-  </joint>
+  <xacro:standoff_rod suffix="1" parent="chassis">
+    <origin xyz="0.075 -0.100 0.1875" rpy="0 0 0" />
+  </xacro:standoff_rod>
+  <xacro:standoff_rod suffix="2" parent="chassis">
+    <origin xyz="-0.075 -0.100 0.1875" rpy="0 0 0" />
+  </xacro:standoff_rod>
+  <xacro:standoff_rod suffix="3" parent="chassis">
+    <origin xyz="-0.075 0.100 0.1875" rpy="0 0 0" />
+  </xacro:standoff_rod>
+  <xacro:standoff_rod suffix="4" parent="chassis">
+    <origin xyz="0.075 0.100 0.1875" rpy="0 0 0" />
+  </xacro:standoff_rod>
   <!-- cup holder tray -->
-  <link name="tray">
-    <visual>
-      <geometry>
-        <cylinder length="${tray_length}" radius="${tray_radius}" />
-      </geometry>
-      <material name="blue" />
-    </visual>
-    <collision>
-      <geometry>
-        <cylinder length="${tray_length}" radius="${tray_radius}" />
-      </geometry>
-    </collision>
-    <inertial>
-      <origin rpy="0 0 0" xyz="0 0 0" />
-      <mass value="${tray_mass}" />
-      <inertia ixx="0.01" iyy="0.01" izz="0.005" ixy="0.0" ixz="0.0" iyz="0.0" />
-    </inertial>
-  </link>
-  <joint name="joint_tray" type="fixed">
-    <origin rpy="0 0 0" xyz="0 0 ${tray_z}" />
-    <parent link="chassis" />
-    <child link="tray" />
-  </joint>
-  <!-- Wheel Left -->
-  <link name="left_wheel">
-    <visual>
-      <origin rpy="0 ${PI/2} ${PI/2}" xyz="0 0 0" />
-      <geometry>
-        <cylinder length="${wheel_length}" radius="${wheel_radius}" />
-      </geometry>
-      <material name="black" />
-    </visual>
-    <collision>
-      <origin rpy="0 ${PI/2} ${PI/2}" xyz="0 0 0" />
-      <geometry>
-        <cylinder length="${wheel_length}" radius="${wheel_radius}" />
-      </geometry>
-    </collision>
-    <inertial>
-      <origin rpy="0 0 0" xyz="0 0 0" />
-      <mass value="${wheel_mass}" />
-      <inertia ixx="0.0001" iyy="0.0001" izz="0.0002" ixy="0.0" ixz="0.0"
-        iyz="0.0" />
-    </inertial>
-  </link>
-  <joint name="joint_left_wheel" type="continuous">
-    <origin rpy="0 0 0" xyz="0 ${wheel_y_offset} ${wheel_z_offset}" />
-    <child link="left_wheel" />
-    <parent link="chassis" />
-    <axis rpy="0 0 0" xyz="0 1 0" />
-    <limit effort="10000" velocity="1000" />
-    <joint_properties damping="1.0" friction="1.0" />
-  </joint>
-  <!-- Wheel Right -->
-  <link name="right_wheel">
-    <visual>
-      <origin rpy="0 ${PI/2} ${PI/2}" xyz="0 0 0" />
-      <geometry>
-        <cylinder length="${wheel_length}" radius="${wheel_radius}" />
-      </geometry>
-      <material name="black" />
-    </visual>
-    <collision>
-      <origin rpy="0 ${PI/2} ${PI/2}" xyz="0 0 0" />
-      <geometry>
-        <cylinder length="${wheel_length}" radius="${wheel_radius}" />
-      </geometry>
-    </collision>
-    <inertial>
-      <origin rpy="0 0 0" xyz="0 0 0" />
-      <mass value="${wheel_mass}" />
-      <inertia ixx="0.0001" iyy="0.0001" izz="0.0002" ixy="0.0" ixz="0.0"
-        iyz="0.0" />
-    </inertial>
-  </link>
-  <joint name="joint_right_wheel" type="continuous">
-    <origin rpy="0 0 0" xyz="0 -${wheel_y_offset} ${wheel_z_offset}" />
-    <child link="right_wheel" />
-    <parent link="chassis" />
-    <axis rpy="0 0 0" xyz="0 1 0" />
-    <limit effort="10000" velocity="1000" />
-    <joint_properties damping="1.0" friction="1.0" />
-  </joint>
-  <!-- front caster Wheel -->
-  <link name="front_caster_wheel">
-    <visual>
-      <origin rpy="0 ${PI/2} ${PI/2}" xyz="0 0 0" />
-      <geometry>
-        <sphere radius="${caster_radius}" />
-      </geometry>
-      <material name="green_dark" />
-    </visual>
-    <collision>
-      <origin rpy="0 ${PI/2} ${PI/2}" xyz="0 0 0" />
-      <geometry>
-        <sphere radius="${caster_radius}" />
-      </geometry>
-    </collision>
-    <inertial>
-      <origin rpy="0 0 0" xyz="0 0 0" />
-      <mass value="0.05" />
-      <inertia ixx="0.0001" iyy="0.0001" izz="0.0001" ixy="0.0" ixz="0.0"
-        iyz="0.0" />
-    </inertial>
-  </link>
-  <joint name="front_pitch_joint" type="continuous">
-    <origin rpy="0 0 0" xyz="${caster_wheel_offset} 0 ${wheel_z_offset}" />
-    <parent link="chassis" />
-    <child link="front_caster_wheel" />
-    <axis xyz="0 1 0" />
-    <limit effort="1000.0" velocity="100.0" />
-    <dynamics damping="0.0" friction="0.1" />
-  </joint>
-  <!-- back caster Wheel -->
-  <link name="back_caster_wheel">
-    <visual>
-      <origin rpy="0 ${PI/2} ${PI/2}" xyz="0 0 0" />
-      <geometry>
-        <sphere radius="${caster_radius}" />
-      </geometry>
-      <material name="green_dark" />
-    </visual>
-    <collision>
-      <origin rpy="0 ${PI/2} ${PI/2}" xyz="0 0 0" />
-      <geometry>
-        <sphere radius="${caster_radius}" />
-      </geometry>
-    </collision>
-    <inertial>
-      <origin rpy="0 0 0" xyz="0 0 0" />
-      <mass value="0.05" />
-      <inertia ixx="0.0001" iyy="0.0001" izz="0.0001" ixy="0.0" ixz="0.0"
-        iyz="0.0" />
-    </inertial>
-  </link>
-  <joint name="back_pitch_joint" type="continuous">
-    <origin rpy="0 0 0" xyz="-${caster_wheel_offset} 0 ${wheel_z_offset}" />
-    <parent link="chassis" />
-    <child link="back_caster_wheel" />
-    <axis xyz="0 1 0" />
-    <limit effort="1000.0" velocity="100.0" />
-    <dynamics damping="0.0" friction="0.1" />
-  </joint>
+  <xacro:cup_holder_tray parent="chassis">
+    <origin xyz="0 0 0.3425" rpy="0 0 0" />
+  </xacro:cup_holder_tray>
+  <xacro:property name="wheel_y_offset" value="0.140" />
+  <xacro:property name="wheel_z_offset" value="-0.0775" />
+  <!-- Wheels -->
+  <xacro:drive_wheel side="left" parent="chassis">
+    <origin xyz="0 0.140 -0.0775" rpy="0 0 0" />
+  </xacro:drive_wheel>
+  <xacro:drive_wheel side="right" parent="chassis">
+    <origin xyz="0 -0.140 -0.0775" rpy="0 0 0" />
+  </xacro:drive_wheel>
+  <!-- caster Wheels -->
+  <xacro:caster_wheel prefix="front" parent="chassis">
+    <origin xyz="0.110 0 -0.0775" rpy="0 0 0" />
+  </xacro:caster_wheel>
+  <xacro:caster_wheel prefix="back" parent="chassis">
+    <origin xyz="-0.110 0 -0.0775" rpy="0 0 0" />
+  </xacro:caster_wheel>
   <!-- Laser model -->
-  <link name="laser_scanner">
-    <visual>
-      <origin rpy="0 0 0" xyz="0 0 -0.0225"/>
-      <geometry>
-        <mesh filename="package://barista_robot_description/meshes/sick_microscan3.dae" scale="0.5 0.5 0.5"/>
-      </geometry>
-    </visual>
-    <collision>
-       <origin rpy="0 0 0" xyz="0 0 0.0204"/>
-      <geometry>
-        <cylinder length="0.0408" radius="0.037493"/>
-      </geometry>
-    </collision>
-    <inertial>
-      <mass value="0.01"/>
-      <origin rpy="0 0 0" xyz="0 0 0.0204"/>
-      <inertia ixx="6.066578520833334e-06" ixy="0" ixz="0" iyy="6.072950163333333e-06" iyz="0" izz="9.365128684166666e-06"/>
-    </inertial>
-  </link>
-  <!-- 0.0775 -->
-  <joint name="joint_laser_scanner" type="continuous">
-    <origin rpy="0 0 0" xyz="${laser_scanner_origin_xy} 0 ${laser_scanner_origin_z}"/>
-    <parent link="chassis"/>
-    <child link="laser_scanner"/>
-    <axis xyz="0 0 1"/>
-    <limit effort="10.0" velocity="2.0"/>
-    <dynamics friction="0.01"/>
-  </joint>
+  <xacro:laser_scanner parent="chassis">
+    <origin xyz="0.12 0 0.14" rpy="0 0 0" />
+  </xacro:laser_scanner>
   <!-- Gazebo materials -->
   <gazebo reference="chassis">

File: xacro/barista_very_simple_main.xacro (robot description, xacro)
@@ -2,4 +2,5 @@
 <robot xmlns:xacro="http://www.ros.org/wiki/xacro" name="barista_bot">
   <xacro:arg name="robot_name" default="barista_X"/>
+  <xacro:property name="robot_name" value="yeyeyea"/>
   <!-- General properties -->
   <xacro:property name="PI" value="3.14159265359"/>
@@ -46,7 +47,7 @@
     <color rgba="${white_color}" />
   </material>
-  <link name="base_link" />
+  <link name="${robot_name}/base_link" />
   <!-- chassis -->
-  <link name="chassis">
+  <link name="${robot_name}/chassis">
     <visual>
       <geometry>
@@ -66,24 +67,24 @@
     </inertial>
   </link>
-  <joint name="base_link_joint" type="fixed">
+  <joint name="${robot_name}/base_link_joint" type="fixed">
     <origin rpy="0 0 0" xyz="0 0 ${base_link_z}" />
-    <parent link="base_link" />
-    <child link="chassis" />
+    <parent link="${robot_name}/base_link" />
+    <child link="${robot_name}/chassis" />
   </joint>
   <!-- standoff rods -->
-  <xacro:standoff_rod suffix="1" parent="chassis">
+  <xacro:standoff_rod suffix="1" parent="${robot_name}/chassis" robot_name="${robot_name}">
     <origin xyz="0.075 -0.100 0.1875" rpy="0 0 0" />
   </xacro:standoff_rod>
-  <xacro:standoff_rod suffix="2" parent="chassis">
+  <xacro:standoff_rod suffix="2" parent="${robot_name}/chassis" robot_name="${robot_name}">
     <origin xyz="-0.075 -0.100 0.1875" rpy="0 0 0" />
   </xacro:standoff_rod>
-  <xacro:standoff_rod suffix="3" parent="chassis">
+  <xacro:standoff_rod suffix="3" parent="${robot_name}/chassis" robot_name="${robot_name}">
     <origin xyz="-0.075 0.100 0.1875" rpy="0 0 0" />
   </xacro:standoff_rod>
-  <xacro:standoff_rod suffix="4" parent="chassis">
+  <xacro:standoff_rod suffix="4" parent="${robot_name}/chassis" robot_name="${robot_name}">
     <origin xyz="0.075 0.100 0.1875" rpy="0 0 0" />
   </xacro:standoff_rod>
   <!-- cup holder tray -->
-  <xacro:cup_holder_tray parent="chassis">
+  <xacro:cup_holder_tray parent="${robot_name}/chassis" robot_name="${robot_name}">
     <origin xyz="0 0 0.3425" rpy="0 0 0" />
   </xacro:cup_holder_tray>
@@ -91,50 +92,50 @@
   <xacro:property name="wheel_z_offset" value="-0.0775" />
   <!-- Wheels -->
-  <xacro:drive_wheel side="left" parent="chassis">
+  <xacro:drive_wheel side="left" parent="${robot_name}/chassis" robot_name="${robot_name}">
     <origin xyz="0 0.140 -0.0775" rpy="0 0 0" />
   </xacro:drive_wheel>
-  <xacro:drive_wheel side="right" parent="chassis">
+  <xacro:drive_wheel side="right" parent="${robot_name}/chassis" robot_name="${robot_name}">
     <origin xyz="0 -0.140 -0.0775" rpy="0 0 0" />
   </xacro:drive_wheel>
   <!-- caster Wheels -->
-  <xacro:caster_wheel prefix="front" parent="chassis">
+  <xacro:caster_wheel prefix="front" parent="${robot_name}/chassis" robot_name="${robot_name}">
     <origin xyz="0.110 0 -0.0775" rpy="0 0 0" />
   </xacro:caster_wheel>
-  <xacro:caster_wheel prefix="back" parent="chassis">
+  <xacro:caster_wheel prefix="back" parent="${robot_name}/chassis" robot_name="${robot_name}">
     <origin xyz="-0.110 0 -0.0775" rpy="0 0 0" />
   </xacro:caster_wheel>
   <!-- Laser model -->
-  <xacro:laser_scanner parent="chassis">
+  <xacro:laser_scanner parent="${robot_name}/chassis">
     <origin xyz="0.12 0 0.14" rpy="0 0 0" />
   </xacro:laser_scanner>
   <!-- Gazebo materials -->
-  <gazebo reference="chassis">
+  <gazebo reference="${robot_name}/chassis">
     <material>Gazebo/Blue</material>
   </gazebo>
-  <gazebo reference="standoff_rod_1">
-    <material>Gazebo/Gray</material>
-  </gazebo>
-  <gazebo reference="standoff_rod_2">
-    <material>Gazebo/Gray</material>
-  </gazebo>
-  <gazebo reference="standoff_rod_3">
-    <material>Gazebo/Gray</material>
-  </gazebo>
-  <gazebo reference="standoff_rod_4">
-    <material>Gazebo/Gray</material>
-  </gazebo>
-  <gazebo reference="tray">
+  <gazebo reference="${robot_name}/standoff_rod_1">
+    <material>Gazebo/Gray</material>
+  </gazebo>
+  <gazebo reference="${robot_name}/standoff_rod_2">
+    <material>Gazebo/Gray</material>
+  </gazebo>
+  <gazebo reference="${robot_name}/standoff_rod_3">
+    <material>Gazebo/Gray</material>
+  </gazebo>
+  <gazebo reference="${robot_name}/standoff_rod_4">
+    <material>Gazebo/Gray</material>
+  </gazebo>
+  <gazebo reference="${robot_name}/tray">
     <material>Gazebo/Blue</material>
   </gazebo>
-  <gazebo reference="left_wheel">
+  <gazebo reference="${robot_name}/left_wheel">
     <material>Gazebo/Black</material>
   </gazebo>
-  <gazebo reference="right_wheel">
+  <gazebo reference="${robot_name}/right_wheel">
     <material>Gazebo/Black</material>
   </gazebo>
-  <gazebo reference="back_caster_wheel">
+  <gazebo reference="${robot_name}/back_caster_wheel">
     <material>Gazebo/Green</material>
   </gazebo>
-  <gazebo reference="front_caster_wheel">
+  <gazebo reference="${robot_name}/front_caster_wheel">
     <material>Gazebo/Green</material>
   </gazebo>
@@ -147,9 +148,9 @@
       </ros>
       <update_rate>30</update_rate>
-      <joint_name>joint_left_wheel</joint_name>
-      <joint_name>joint_right_wheel</joint_name>
-      <joint_name>front_pitch_joint</joint_name>
-      <joint_name>back_pitch_joint</joint_name>
-      <joint_name>joint_laser_scanner</joint_name>
+      <joint_name>${robot_name}/joint_left_wheel</joint_name>
+      <joint_name>${robot_name}/joint_right_wheel</joint_name>
+      <joint_name>${robot_name}/front_pitch_joint</joint_name>
+      <joint_name>${robot_name}/back_pitch_joint</joint_name>
+      <joint_name>${robot_name}/joint_laser_scanner</joint_name>
     </plugin>
   </gazebo>
@@ -158,6 +159,6 @@
     <plugin filename="libgazebo_ros_diff_drive.so" name="differential_drive_controller">
       <!-- wheels -->
-      <left_joint>joint_left_wheel</left_joint>
-      <right_joint>joint_right_wheel</right_joint>
+      <left_joint>${robot_name}/joint_left_wheel</left_joint>
+      <right_joint>${robot_name}/joint_right_wheel</right_joint>
       <!-- kinematics -->
       <wheel_separation>0.1</wheel_separation>
@@ -169,9 +170,9 @@
       <publish_odom>true</publish_odom>
       <publish_odom_tf>true</publish_odom_tf>
-      <odometry_frame>odom</odometry_frame>
-      <robot_base_frame>base_link</robot_base_frame>
+      <odometry_frame>${robot_name}/odom</odometry_frame>
+      <robot_base_frame>${robot_name}/base_link</robot_base_frame>
     </plugin>
   </gazebo>
-  <gazebo reference="laser_scanner">
+  <gazebo reference="${robot_name}/laser_scanner">
     <sensor name="sensor_ray" type="ray">
         <pose>0 0 0 0 0 0</pose>
@@ -195,5 +196,6 @@
         <plugin name="laser" filename="libgazebo_ros_ray_sensor.so">
           <ros>
-            <remapping>~/out:=scan</remapping>
+            <namespace>/${robot_name}</namespace>
+            <remapping>~/out:=/thescan</remapping>
           </ros>
           <output_type>sensor_msgs/LaserScan</output_type>

File: xacro/caster_wheel.xacro (robot description, xacro)
@@ -6,6 +6,6 @@
   <xacro:property name="caster_mass" value="0.05" />
   <xacro:property name="M_PI" value="3.14159265359" />
-  <xacro:macro name="caster_wheel" params="prefix parent *origin">
-    <link name="${prefix}_caster_wheel">
+  <xacro:macro name="caster_wheel" params="prefix parent robot_name *origin">
+    <link name="${robot_name}/${prefix}_caster_wheel">
       <visual>
         <origin rpy="0 ${M_PI/2} ${M_PI/2}" xyz="0 0 0" />
@@ -33,8 +33,8 @@
       </inertial>
     </link>
-    <joint name="${prefix}_pitch_joint" type="continuous">
+    <joint name="${robot_name}/${prefix}_pitch_joint" type="continuous">
       <xacro:insert_block name="origin" />
       <parent link="${parent}" />
-      <child link="${prefix}_caster_wheel" />
+      <child link="${robot_name}/${prefix}_caster_wheel" />
       <axis xyz="0 1 0" />
       <limit effort="1000.0" velocity="100.0" />

File: xacro/cup_holder_tray.xacro (robot description, xacro)
@@ -6,6 +6,6 @@
   <xacro:property name="tray_radius" value="0.160" />
   <xacro:property name="tray_mass" value="0.5" />
-  <xacro:macro name="cup_holder_tray" params="parent *origin">
-    <link name="tray">
+  <xacro:macro name="cup_holder_tray" params="parent robot_name *origin">
+    <link name="${robot_name}/tray">
       <visual>
         <geometry>
@@ -31,8 +31,8 @@
       </inertial>
     </link>
-    <joint name="joint_tray" type="fixed">
+    <joint name="${robot_name}/joint_tray" type="fixed">
       <xacro:insert_block name="origin" />
       <parent link="${parent}" />
-      <child link="tray" />
+      <child link="${robot_name}/tray" />
     </joint>
   </xacro:macro>

File: xacro/drive_wheel.xacro (robot description, xacro)
@@ -7,6 +7,6 @@
   <xacro:property name="wheel_mass" value="0.2" />
   <xacro:property name="M_PI" value="3.14159265359" />
-  <xacro:macro name="drive_wheel" params="side parent *origin">
-    <link name="${side}_wheel">
+  <xacro:macro name="drive_wheel" params="side parent robot_name *origin">
+    <link name="${robot_name}/${side}_wheel">
       <visual>
         <origin rpy="0 ${M_PI/2} ${M_PI/2}" xyz="0 0 0" />
@@ -34,7 +34,7 @@
       </inertial>
     </link>
-    <joint name="joint_${side}_wheel" type="continuous">
+    <joint name="${robot_name}/joint_${side}_wheel" type="continuous">
       <xacro:insert_block name="origin" />
-      <child link="${side}_wheel" />
+      <child link="${robot_name}/${side}_wheel" />
       <parent link="${parent}" />
       <axis rpy="0 0 0" xyz="0 1 0" />
