Commit message: returned to 1 robot spawn but with manually putting namespace before every frame and robot_description topic

File: xacro/laser_scanner.xacro (robot description, xacro)
@@ -9,5 +9,5 @@
   <xacro:macro name="laser_scanner" params="parent *origin">
     <xacro:if value="${include_laser}">
-      <link name="laser_scanner">
+      <link name="${robot_name}/laser_scanner">
         <visual>
           <origin rpy="0 0 0" xyz="0 0 -0.062" />
@@ -36,8 +36,8 @@
         </inertial>
       </link>
-      <joint name="joint_laser_scanner" type="continuous">
+      <joint name="${robot_name}/joint_laser_scanner" type="continuous">
         <xacro:insert_block name="origin" />
         <parent link="${parent}" />
-        <child link="laser_scanner" />
+        <child link="${robot_name}/laser_scanner" />
         <axis xyz="0 0 1" />
         <limit effort="10.0" velocity="2.0" />

File: xacro/standoff_rod.xacro (robot description, xacro)
@@ -6,6 +6,6 @@
   <xacro:property name="rod_radius" value="0.010" />
   <xacro:property name="rod_mass" value="0.1" />
-  <xacro:macro name="standoff_rod" params="suffix parent *origin">
-    <link name="standoff_rod_${suffix}">
+  <xacro:macro name="standoff_rod" params="suffix parent robot_name *origin">
+    <link name="${robot_name}/standoff_rod_${suffix}">
       <visual>
         <geometry>
@@ -31,8 +31,8 @@
       </inertial>
     </link>
-    <joint name="joint_standoff_rod_${suffix}" type="fixed">
+    <joint name="${robot_name}/joint_standoff_rod_${suffix}" type="fixed">
       <xacro:insert_block name="origin" />
       <parent link="${parent}" />
-      <child link="standoff_rod_${suffix}" />
+      <child link="${robot_name}/standoff_rod_${suffix}" />
     </joint>
   </xacro:macro>
