Commit message: Succesfully spawn 2 robots properly namespaced!

File: xacro/barista_very_simple_main.xacro (robot description, xacro)
@@ -1,6 +1,7 @@
 <?xml version="1.0"?>
 <robot xmlns:xacro="http://www.ros.org/wiki/xacro" name="barista_bot">
-  <xacro:arg name="robot_name" default="barista_X"/>
-  <xacro:property name="robot_name" value="yeyeyea"/>
+  <!-- <xacro:arg name="robot_name_arg" default="PROUTPIPI"/> -->
+  <xacro:property name="robot_name" value="default_name" />
+  <xacro:property name="robot_name" value="$(arg robot_name_arg)"/>
   <!-- General properties -->
   <xacro:property name="PI" value="3.14159265359"/>
@@ -47,4 +48,5 @@
     <color rgba="${white_color}" />
   </material>
+  <!-- base_link -->
   <link name="${robot_name}/base_link" />
   <!-- chassis -->
@@ -143,8 +145,9 @@
   <!-- JOINT PUBLISHER -->
   <gazebo>
-    <plugin name="box_bot_joint_state" filename="libgazebo_ros_joint_state_publisher.so">
-      <ros>
+    <plugin name="${robot_name}_joint_state" filename="libgazebo_ros_joint_state_publisher.so">
+        <ros>
+          <namespace>/${robot_name}</namespace> <!-- ADD NAMESPACE -->
           <remapping>~/out:=joint_states</remapping>
-      </ros>
+        </ros>
       <update_rate>30</update_rate>
       <joint_name>${robot_name}/joint_left_wheel</joint_name>
@@ -157,5 +160,8 @@
   <!-- Differential drive -->
   <gazebo>
-    <plugin filename="libgazebo_ros_diff_drive.so" name="differential_drive_controller">
+    <plugin filename="libgazebo_ros_diff_drive.so" name="${robot_name}_differential_drive_controller" >
+      <ros>
+        <namespace>/${robot_name}</namespace> <!-- ADD NAMESPACE -->
+      </ros>
       <!-- wheels -->
       <left_joint>${robot_name}/joint_left_wheel</left_joint>
@@ -196,6 +202,6 @@
         <plugin name="laser" filename="libgazebo_ros_ray_sensor.so">
           <ros>
-            <namespace>/${robot_name}</namespace>
-            <remapping>~/out:=/thescan</remapping>
+            <namespace>/${robot_name}</namespace> <!-- Already had this -->
+            <remapping>~/out:=scan</remapping> <!-- Changed topic name -->
           </ros>
           <output_type>sensor_msgs/LaserScan</output_type>
